File: Garuda_PCB/Payloadv03.brd (EAGLE design)
At the start: 80.8 x 155.8 mm, 32 parts, among them IC1 7805TV, IC2 LM1117T-3.3-V, Q2 IRF540, U1 GY-521MPU6050

Commit message: routed pcb v03
Parts:
- moved AIRSPEED_SENSOR 63.8 mm to (-29.2, 115.6), turned to 0 degrees
- moved SERVO 55.0 mm to (-24.1, 109.2), turned to 180 degrees
- moved C2 3.81 mm to (2.54, 128.3)
- moved XB1 3.71 mm to (23.0, 107.0), turned to 189.6 degrees
- moved IC2 2.84 mm to (27.9, 135.9)
- moved C1 2.54 mm to (2.54, 134.6)
- moved C3 1.27 mm to (11.4, 133.3)
- moved IC1 1.27 mm to (11.3, 140.4)
- moved JUMPER3 1.27 mm to (12.7, 123.2)
- moved C4 1.27 mm to (11.4, 128.3)
Connections:
- removed net AGND: U$2.AGND
- removed net ENBLUE: U$2.20/A6
- removed net HALLIP: U$2.5
- removed net RXBLUE: U$2.10
- removed net TXBLUE: U$2.9
- net GND: now also U$2.AGND
- net RXGPS: now also U$2.7
- net RX_PM2.5: now also U$2.10; no longer U$2.8
- net SERVO: now also U$2.21/A7
- net SPEED_DATA: now also U$2.23/A9
- net TXGPS: now also U$2.8
- net TX_PM2.5: now also U$2.9; no longer U$2.7
Routing:
- net GND: track 0.00 -> 328.8 mm
- net 5VOUT: track 0.00 -> 153.7 mm
- net 3.3VOUT: track 0.00 -> 129.7 mm
- net 12V: track 0.00 -> 92.8 mm
- net 9V: track 0.00 -> 87.1 mm
- net BUZZER: track 0.00 -> 77.0 mm
- net RXGPS: track 0.00 -> 75.0 mm
- net TXGPS: track 0.00 -> 66.1 mm
- net SCL: track 0.00 -> 65.1 mm, vias 0 -> 1
- net SDA: track 0.00 -> 63.1 mm
- net ENGPS: track 0.00 -> 56.5 mm
- net SCK: track 0.00 -> 40.6 mm
- net 3.3VTEENSY: track 0.00 -> 32.3 mm
- net N$3: track 0.00 -> 29.4 mm
- net TX_PM2.5: track 0.00 -> 23.8 mm
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