File: Garuda_PCB/Payloadv03.sch (EAGLE design)
At the start: 29 parts, among them IC1 7805TV, IC2 LM1117T-3.3-V, Q2 IRF540, U1 GY-521MPU6050

Commit message: routed pcb v03
Parts:
- added AIRSPEED_SENSOR, SERVO: 455-1750-1-ND, SparkFun-Connectors:CONN_03
- added PM2.5: (no value), SparkFun-Connectors:CONN_04
Connections:
- removed net 3.3V_TEENSY: JUMPER1.1
- removed net ENBLUE: U$2.20/A6/PWM
- removed net HALLIP: U$2.5/PWM
- removed net RXBLUE: U$2.10/TX2/PWM
- removed net TXBLUE: U$2.9/RX2/PWM
- new net RX_PM2.5: PM2.5.3, U$2.10/TX2/PWM
- new net SERVO: SERVO.1, U$2.21/A7/PWM
- new net SPEED_DATA: AIRSPEED_SENSOR.2, U$2.23/A9/T/PWM
- new net TX_PM2.5: PM2.5.2, U$2.9/RX2/PWM
- net 3.3VIN: no longer BMP280.1, BMP280.6, U1.ADO
- net 3.3VOUT: now also BMP280.1, BMP280.6, U1.ADO, XB1.VCC
- net 3.3VTEENSY: now also JUMPER1.1
- net 5VOUT: now also AIRSPEED_SENSOR.3, PM2.5.4, SERVO.2
- net GND: now also AIRSPEED_SENSOR.1, PM2.5.1, SERVO.3, U$2.AGND
- net RXGPS: now also U$2.7/RX3; no longer U$2.8/TX3
- net TXGPS: now also U$2.8/TX3; no longer U$2.7/RX3
